File: RPU-2 [Aquila]/KiCAD/REDS/REDS.kicad_sch (KiCad schematic)
At the start: 15 parts, among them J1 Pigtail, J2 Our Power, M1 Motor_Servo, U2 AmazonBuck, U3 LM555xN, U4 MAX4544

Commit message: Changed the set up to 1uF Cap
Parts:
- C1: value 100nF -> 1uF
- R2: value 16k -> 2.2k
- R4: value 20k -> 1k
Changed lines of the file:
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@@
 			)
 		)
-		(property "Value" "20k"
+		(property "Value" "1k"
 			(at 102.87 53.3399 0)
 			(show_name no)
@@
 			)
 		)
-		(property "Value" "16k"
+		(property "Value" "2.2k"
 			(at 102.87 66.0399 90)
 			(show_name no)
@@
 			)
 		)
-		(property "Value" "100nF"
+		(property "Value" "1uF"
 			(at 147.32 85.0962 0)
 			(show_name no)
