File: RPU-2 [Aquila]/KiCAD/REDS/REDS.kicad_sch (KiCad schematic)
At the start: 15 parts, among them J1 Pigtail, J2 Our Power, M1 Motor_Servo, U2 AmazonBuck, U3 LM555xN, U4 MAX4544

Commit message: schem
Parts:
- removed J2: Our Power, Connector_Wire:SolderWire-0.15sqmm_1x02_P4mm_D0.5mm_OD1.5mm, symbol Connector:Screw_Terminal_01x02
- added J3: Reds Power, Connector_Wire:SolderWire-0.15sqmm_1x02_P4mm_D0.5mm_OD1.5mm, symbol Connector:Screw_Terminal_01x02
- added J4: Screw_Terminal_01x03, Connector_Wire:SolderWire-0.15sqmm_1x03_P4mm_D0.5mm_OD1.5mm, symbol Connector:Screw_Terminal_01x03
- J1: footprint Connector_Wire:SolderWire-0.15sqmm_1x02_P4mm_D0.5mm_OD1.5mm -> (none)
- R2: value 16k -> 1.5k
- R4: value 20k -> 1.8k
- U2: footprint Package_SO:SOIC-8_3.9x4.9mm_P1.27mm -> (none)
- U4: footprint Package_SO:MSOP-8_3x3mm_P0.65mm -> Package_DIP:DIP-8_W7.62mm
Connections:
- net +6.8V: now also J3.1 (Pin_1)
- net GND: now also J3.2 (Pin_2), J4.1 (Pin_1)
- net OurPower: now also J4.2 (Pin_2)
- net OurSignal: now also J4.3 (Pin_3)
